Commit message: Add Ubuntu 22.04 and ROS 2 Humble support
Port MoveIt, Servo, Gazebo, and teleoperation launch paths to Humble; add the reusable MTC waypoint sequence and replay service; and include corrected robot and optional suction-tool geometry.

File: src/igus_rebel_description/urdf/igus_rebel2.control.xacro (robot description, xacro)
@@ -5,5 +5,5 @@
         <xacro:macro name="joint_control" params="joint">
             <joint name="${joint}">
-                <xacro:if value="${hardware_protocol == 'gazebo'}">
+                <xacro:if value="${hardware_protocol == 'gazebo' or hardware_protocol == 'isaac_topic' or hardware_protocol == 'mock_hardware'}">
                     <command_interface name="position" />
                 </xacro:if>
@@ -22,4 +22,10 @@
                 <xacro:if value="${hardware_protocol == 'gazebo'}">
                     <plugin>gz_ros2_control/GazeboSimSystem</plugin>
+                </xacro:if>
+                <xacro:if value="${hardware_protocol == 'isaac_topic'}">
+                    <plugin>topic_based_ros2_control/TopicBasedSystem</plugin>
+                    <param name="joint_commands_topic">/isaac_joint_commands</param>
+                    <param name="joint_states_topic">/isaac_joint_states</param>
+                    <param name="trigger_joint_command_threshold">0.0001</param>
                 </xacro:if>
                 <xacro:if value="${hardware_protocol == 'rebel'}">

File: src/igus_rebel_description/urdf/igus_rebel2_robotviewer.urdf (robot description, URDF)
Before this commit: robot igus_rebel, 12 links, 11 joints
Links:
- link base_link: geometry collision cylinder length=0.1 radius=0.09; visual mesh filename=package://igus_rebel_description/meshes/rebel_d00617809/bas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
- link link1: geometry collision box size=0.1 0.03 0.1; visual mesh filename=package://igus_rebel_description/meshes/rebel_d00617809/lin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
- link link2: geometry collision cylinder length=0.18 radius=0.06; visual mesh filename=package://igus_rebel_description/meshes/rebel_d00617809/lin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
- link link3: geometry collision box size=0.1 0.03 0.1; visual mesh filename=package://igus_rebel_description/meshes/rebel_d00617809/lin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
- link link4: geometry collision cylinder length=0.1 radius=0.05; visual mesh filename=package://igus_rebel_description/meshes/rebel_d00617809/lin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
- link link5: geometry collision box size=0.1 0.03 0.1; visual mesh filename=package://igus_rebel_description/meshes/rebel_d00617809/lin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
- link link6: geometry collision cylinder length=0.065 radius=0.04; visual mesh filename=package://igus_rebel_description/meshes/rebel_d00617809/lin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
- link motor1: geometry collision cylinder length=0.065 radius=0.05; visual mesh filename=package://igus_rebel_description/meshes/rebel_d00617809/mot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
- link motor2: geometry collision cylinder length=0.065 radius=0.05; visual mesh filename=package://igus_rebel_description/meshes/rebel_d00617809/mot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
- link motor3: geometry collision cylinder length=0.065 radius=0.05; visual mesh filename=package://igus_rebel_description/meshes/rebel_d00617809/mot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
- link motor4: geometry collision cylinder length=0.065 radius=0.05; visual mesh filename=package://igus_rebel_description/meshes/rebel_d00617809/mot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
- link motor5: geometry collision cylinder length=0.065 radius=0.04; visual mesh filename=package://igus_rebel_description/meshes/rebel_d00617809/mot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
