Commit message: Make CRI controller address configurable, default wired LAN 192.168.3.11
The driver reads ros2_control hardware parameters robot_ip/robot_port
(validated; invalid values make on_init fail before connecting). The
xacro wrapper and rebel.launch.py expose robot_ip, defaulting to the
wired LAN address 192.168.3.11; Wi-Fi uses robot_ip:=192.168.50.133.
Adds unit tests for the default, the override and invalid values.

Co-Authored-By: Claude Opus 5.5 <noreply@anthropic.com>

File: src/igus_rebel_description/urdf/igus_rebel2.control.xacro (robot description, xacro)
@@ -2,5 +2,5 @@
 <!-- igus_rebel.control.xacro -->
 <robot xmlns:xacro="http://www.ros.org/wiki/xacro">
-    <xacro:macro name="igus_rebel_control" params="arm_id hardware_protocol">
+    <xacro:macro name="igus_rebel_control" params="arm_id hardware_protocol robot_ip:=192.168.3.11 robot_port:=3920">
         <xacro:macro name="joint_control" params="joint">
             <joint name="${joint}">
@@ -31,4 +31,6 @@
                 <xacro:if value="${hardware_protocol == 'rebel'}">
                     <plugin>Igus/Rebel</plugin>
+                    <param name="robot_ip">${robot_ip}</param>
+                    <param name="robot_port">${robot_port}</param>
                 </xacro:if>
             </hardware>

File: src/igus_rebel_description/urdf/igus_rebel_xeg32_wrapper.urdf.xacro (robot description, xacro)
@@ -4,4 +4,6 @@
   <!-- Keep the ReBeL arm hardware configuration independent from the gripper. -->
   <xacro:arg name="hardware_protocol" default="rebel"/>
+  <!-- CRI controller address: 192.168.3.11 = wired LAN (default), 192.168.50.133 = Wi-Fi. -->
+  <xacro:arg name="robot_ip" default="192.168.3.11"/>
   <xacro:arg name="include_ros2_control" default="true"/>
   <xacro:arg name="attach_xeg32" default="true"/>
@@ -15,5 +17,6 @@
     <xacro:igus_rebel_control
       arm_id="rebel_arm"
-      hardware_protocol="$(arg hardware_protocol)"/>
+      hardware_protocol="$(arg hardware_protocol)"
+      robot_ip="$(arg robot_ip)"/>
   </xacro:if>
   <!-- Same world attachment used by igus_rebel_robot2.urdf.xacro. -->
