Commit message: Integrate external vision planning workflow

File: src/igus_rebel_description/urdf/igus_rebel_xeg32_wrapper.urdf.xacro (robot description, xacro)
@@ -6,18 +6,7 @@
   <xacro:arg name="include_ros2_control" default="true"/>
   <xacro:arg name="attach_xeg32" default="true"/>
-  <!--
-    Fixed hardware mount, verified from the assembled XEG model. The gripper
-    itself is never moved by a knife-pose experiment. The 25 x 25 mm knife is
-    gripped at its CAD-verified jaw position; candidate poses may only change
-    the knife transform while retaining a physically valid jaw engagement.
-  -->
+  <!-- Retained rough gripper mount; not used to define the calibrated TCP. -->
   <xacro:arg name="xeg32_mount_xyz" default="0 0 0.052"/>
   <xacro:arg name="xeg32_mount_rpy" default="0 0 0.261799"/>
-  <xacro:arg name="attach_cutter" default="true"/>
-  <xacro:arg name="cutter_mount_xyz" default="-0.077 0 0.029"/>
-  <xacro:arg name="cutter_mount_rpy" default="0 0 0"/>
-  <xacro:arg name="cutter_length" default="0.1855"/>
-  <xacro:arg name="cutter_width" default="0.025"/>
-  <xacro:arg name="cutter_tip_length" default="0.015"/>
   <xacro:include filename="$(find igus_rebel_description)/urdf/igus_rebel2.urdf"/>
   <xacro:include filename="$(find igus_rebel_description)/urdf/igus_rebel2.control.xacro"/>
@@ -40,11 +29,26 @@
       prefix="xeg32_"
       flange_xyz="$(arg xeg32_mount_xyz)"
-      flange_rpy="$(arg xeg32_mount_rpy)"
-      attach_cutter="$(arg attach_cutter)"
-      cutter_mount_xyz="$(arg cutter_mount_xyz)"
-      cutter_mount_rpy="$(arg cutter_mount_rpy)"
-      cutter_length="$(arg cutter_length)"
-      cutter_width="$(arg cutter_width)"
-      cutter_tip_length="$(arg cutter_tip_length)"/>
+      flange_rpy="$(arg xeg32_mount_rpy)"/>
   </xacro:if>
+  <!-- Calibrated frames remain available even when gripper visuals are omitted. -->
+  <link name="igus_tool0"/>
+  <joint name="link6_to_igus_tool0" type="fixed">
+    <parent link="link6"/>
+    <child link="igus_tool0"/>
+    <origin xyz="0 0 0.0527" rpy="0 0 3.141592653589793"/>
+  </joint>
+  <link name="xeg32_tool_tip">
+    <visual>
+      <geometry><sphere radius="0.006"/></geometry>
+      <material name="xeg32_tool_tip_marker"><color rgba="0.1 1 0.1 1"/></material>
+    </visual>
+    <!-- Tip-only proxy: does not cover the attached cutter body. -->
+    <collision><geometry><sphere radius="0.006"/></geometry></collision>
+  </link>
+  <joint name="igus_tool0_to_xeg32_tool_tip" type="fixed">
+    <parent link="igus_tool0"/>
+    <child link="xeg32_tool_tip"/>
+    <!-- knivetool4_with_pose2 XML OFFSET, converted from millimetres to metres. -->
+    <origin xyz="0.068936 0.046766 0.127060" rpy="0 0 0"/>
+  </joint>
 </robot>

File: src/igus_rebel_description/urdf/xeg32_gripper.urdf.xacro (robot description, xacro)
@@ -1,6 +1,6 @@
 <?xml version='1.0' encoding='utf-8'?>
 <robot xmlns:xacro="http://www.ros.org/wiki/xacro">
-  <!-- Reusable HIWIN XEG-32 gripper + camera-mount macro. Geometry/kinematics are taken from the latest Onshape export. -->
-  <xacro:macro name="xeg32_gripper" params="parent_link prefix flange_xyz flange_rpy lock_joints:=true attach_cutter:=true cutter_mount_xyz:='-0.077 0 0.029' cutter_mount_rpy:='0 0 0' cutter_length:=0.1855 cutter_width:=0.025 cutter_tip_length:=0.015">
+  <!-- Rough HIWIN XEG-32 gripper and camera-mount geometry; independent of TCP calibration. -->
+  <xacro:macro name="xeg32_gripper" params="parent_link prefix flange_xyz flange_rpy lock_joints:=true">
     <joint name="${prefix}mount_joint" type="fixed">
       <origin xyz="${flange_xyz}" rpy="${flange_rpy}" />
@@ -60,57 +60,4 @@
       </collision>
     </link>
-    <!-- Plan-only knife: 185.5 mm overall, 25 x 25 mm body, and a 15 mm square-pyramid tip. -->
-    <xacro:if value="${attach_cutter}">
-      <joint name="${prefix}cutter_mount_joint" type="fixed">
-        <origin xyz="${cutter_mount_xyz}" rpy="${cutter_mount_rpy}" />
-        <parent link="${prefix}base_link" />
-        <child link="${prefix}cutter_link" />
-      </joint>
-      <link name="${prefix}cutter_link">
-        <visual>
-          <origin xyz="0 0 ${-cutter_tip_length / 2.0}" rpy="0 0 0" />
-          <geometry>
-            <box size="${cutter_width} ${cutter_width} ${cutter_length - cutter_tip_length}" />
-          </geometry>
-          <material name="${prefix}cutter_material">
-            <color rgba="0.85 0.15 0.15 1" />
-          </material>
-        </visual>
-        <collision>
-          <origin xyz="0 0 ${-cutter_tip_length / 2.0}" rpy="0 0 0" />
-          <geometry>
-            <box size="${cutter_width} ${cutter_width} ${cutter_length - cutter_tip_length}" />
-          </geometry>
-        </collision>
-        <visual>
-          <origin xyz="0 0 ${cutter_length / 2.0 - cutter_tip_length / 2.0}" rpy="0 0 0" />
-          <geometry>
-            <mesh filename="package://igus_rebel_description/meshes/xeg32/cutter_tip_15mm.stl" />
-          </geometry>
-          <material name="${prefix}cutter_tip_material">
-            <color rgba="0.75 0.78 0.82 1" />
-          </material>
-        </visual>
-        <collision>
-          <origin xyz="0 0 ${cutter_length / 2.0 - cutter_tip_length / 2.0}" rpy="0 0 0" />
-          <geometry>
-            <mesh filename="package://igus_rebel_description/meshes/xeg32/cutter_tip_15mm.stl" />
-          </geometry>
-        </collision>
-      </link>
-      <joint name="${prefix}tool_tip_joint" type="fixed">
-        <!-- Calibrated against the saved middle_only seam_end target 1788412047_726417920. -->
-        <origin xyz="-0.012644 -0.004722 0.082408" rpy="0 0 0" />
-        <parent link="${prefix}cutter_link" />
-        <child link="${prefix}tool_tip" />
-      </joint>
-      <!-- Visual-only TCP locator: the physical knife geometry remains unchanged. -->
-      <link name="${prefix}tool_tip">
-        <visual>
-          <geometry><sphere radius="0.006" /></geometry>
-          <material name="${prefix}tool_tip_marker"><color rgba="0.1 1 0.1 1" /></material>
-        </visual>
-      </link>
-    </xacro:if>
     <link name="${prefix}left_carriage_link">
       <inertial>
