Commit message: Add H-cut wrist guard, transit planner, and XEG-32 assets
- box_h_cut_executor: joint-interpolation-first free-space transit
  planner, separate transit scalings (default 0.05), and a fail-closed
  check rejecting free-space transits with joint6 travel > pi.
- Collision-aware left learned-orientation IK with carton and external
  camera-pole collision object.
- XEG-32 collision meshes,
  TCP GUI package, table cloud filter, SetCartesianIncrement srv.
- HANDOFF.md documenting mock-only verification state. The corrected
  (old left teaching) T-cut is still rejected by the wrist guard;
  nothing here is validated on the physical robot.

Co-Authored-By: Claude Opus 5.5 <noreply@anthropic.com>

File: src/igus_rebel_description/urdf/igus_rebel_xeg32_wrapper.urdf.xacro (robot description, xacro)
@@ -43,12 +43,21 @@
       <material name="xeg32_tool_tip_marker"><color rgba="0.1 1 0.1 1"/></material>
     </visual>
-    <!-- Tip-only proxy: does not cover the attached cutter body. -->
-    <collision><geometry><sphere radius="0.006"/></geometry></collision>
   </link>
+  <!-- touch-corrected 2026-09-24c: XY-only safety fix (tip -0.7/+4.6mm tool from CENTER residual); Z held at +15mm fix (0.130699) pending stale-model check -->
   <joint name="igus_tool0_to_xeg32_tool_tip" type="fixed">
     <parent link="igus_tool0"/>
     <child link="xeg32_tool_tip"/>
-    <!-- knivetool4_with_pose2 XML OFFSET, converted from millimetres to metres. -->
-    <origin xyz="0.068936 0.046766 0.127060" rpy="0 0 0"/>
+    <origin xyz="0.005937 0.094121 0.130699" rpy="0 0 0"/>
+  </joint>
+  <link name="xeg32_tool_tip_proposed">
+    <visual>
+      <geometry><sphere radius="0.006"/></geometry>
+      <material name="xeg32_tool_tip_proposed_marker"><color rgba="1 0.1 0.1 1"/></material>
+    </visual>
+  </link>
+  <joint name="igus_tool0_to_xeg32_tool_tip_proposed" type="fixed">
+    <parent link="igus_tool0"/>
+    <child link="xeg32_tool_tip_proposed"/>
+    <origin xyz="0.088936 0.046766 0.135060" rpy="0 0 0"/>
   </joint>
 </robot>

File: src/igus_rebel_description/urdf/xeg32_gripper.urdf.xacro (robot description, xacro)
@@ -1,5 +1,5 @@
 <?xml version='1.0' encoding='utf-8'?>
 <robot xmlns:xacro="http://www.ros.org/wiki/xacro">
-  <!-- Rough HIWIN XEG-32 gripper and camera-mount geometry; independent of TCP calibration. -->
+  <!-- Rough HIWIN XEG-32 gripper geometry; independent of TCP calibration. -->
   <xacro:macro name="xeg32_gripper" params="parent_link prefix flange_xyz flange_rpy lock_joints:=true">
     <joint name="${prefix}mount_joint" type="fixed">
@@ -26,5 +26,5 @@
         <origin xyz="0.049 -0 0.016" rpy="0 -0 -1.5708" />
         <geometry>
-          <mesh filename="package://igus_rebel_description/meshes/xeg32/part_1.stl" />
+          <mesh filename="package://igus_rebel_description/meshes/xeg32_collision/part_1.stl" />
         </geometry>
       </collision>
@@ -41,5 +41,5 @@
         <origin xyz="0.0065 -0 0.029" rpy="0 -0 -1.5708" />
         <geometry>
-          <mesh filename="package://igus_rebel_description/meshes/xeg32/xeg_base.stl" />
+          <mesh filename="package://igus_rebel_description/meshes/xeg32_collision/xeg_base.stl" />
         </geometry>
       </collision>
@@ -56,5 +56,5 @@
         <origin xyz="0 0 0" rpy="0 0 -1.5708" />
         <geometry>
-          <mesh filename="package://igus_rebel_description/meshes/xeg32/part_1__2.stl" />
+          <mesh filename="package://igus_rebel_description/meshes/xeg32_collision/part_1__2.stl" />
         </geometry>
       </collision>
@@ -93,5 +93,5 @@
         <origin xyz="-2.30037e-07 -0.004 -0.00315591" rpy="-1.5708 0 0" />
         <geometry>
-          <mesh filename="package://igus_rebel_description/meshes/xeg32/part_1__3.stl" />
+          <mesh filename="package://igus_rebel_description/meshes/xeg32_collision/part_1__3.stl" />
         </geometry>
       </collision>
@@ -115,5 +115,5 @@
         <origin xyz="-2.30037e-07 -0.004 -0.00315591" rpy="-1.5708 0 -0" />
         <geometry>
-          <mesh filename="package://igus_rebel_description/meshes/xeg32/part_1__3.stl" />
+          <mesh filename="package://igus_rebel_description/meshes/xeg32_collision/part_1__3.stl" />
         </geometry>
       </collision>
@@ -134,41 +134,4 @@
       </collision>
     </link>
-    <link name="${prefix}camera_mount_link">
-      <inertial>
-        <origin xyz="0 0 0" rpy="0 0 0" />
-        <mass value="1e-09" />
-        <inertia ixx="1e-09" ixy="0" ixz="0" iyy="1e-09" iyz="0" izz="1e-09" />
-      </inertial>
-      <visual>
-        <origin xyz="-0.0120767 0.0750311 -0.0273242" rpy="1e-12 -1.56937 -1.5708" />
-        <geometry>
-          <mesh filename="package://igus_rebel_description/meshes/xeg32/00_mb2502_asm_1_1.stl" />
-        </geometry>
-        <material name="${prefix}00_mb2502_asm_1_1_material">
-          <color rgba="0.917647 0.917647 0.917647 1" />
-        </material>
-      </visual>
-      <collision>
-        <origin xyz="-0.0120767 0.0750311 -0.0273242" rpy="1e-12 -1.56937 -1.5708" />
-        <geometry>
-          <mesh filename="package://igus_rebel_description/meshes/xeg32/00_mb2502_asm_1_1.stl" />
-        </geometry>
-      </collision>
-      <visual>
-        <origin xyz="0 0.032 -0.009" rpy="-1.5708 -1.5708 0" />
-        <geometry>
-          <mesh filename="package://igus_rebel_description/meshes/xeg32/part_1__4.stl" />
-        </geometry>
-        <material name="${prefix}part_1_5_material">
-          <color rgba="0.647059 0.647059 0.647059 1" />
-        </material>
-      </visual>
-      <collision>
-        <origin xyz="0 0.032 -0.009" rpy="-1.5708 -1.5708 0" />
-        <geometry>
-          <mesh filename="package://igus_rebel_description/meshes/xeg32/part_1__4.stl" />
-        </geometry>
-      </collision>
-    </link>
     <!-- The ReBeL driver currently publishes arm states only. Lock the
          unactuated XEG joints in the planning model until a gripper controller
@@ -184,9 +147,4 @@
         <parent link="${prefix}base_link" />
         <child link="${prefix}right_carriage_link" />
-      </joint>
-      <joint name="${prefix}camera_tilt_joint" type="fixed">
-        <origin xyz="0.071 -0.0092 0.055" rpy="1.5708 -0.149605 -0" />
-        <parent link="${prefix}base_link" />
-        <child link="${prefix}camera_mount_link" />
       </joint>
     </xacro:if>
@@ -207,11 +165,4 @@
         <mimic joint="${prefix}left_carriage_joint" multiplier="1.0" />
       </joint>
-      <joint name="${prefix}camera_tilt_joint" type="revolute">
-        <origin xyz="0.071 -0.0092 0.055" rpy="1.5708 -0.149605 -0" />
-        <parent link="${prefix}base_link" />
-        <child link="${prefix}camera_mount_link" />
-        <axis xyz="0 0 1" />
-        <limit effort="10" velocity="10" lower="-0.062339" upper="0.373993" />
-      </joint>
     </xacro:unless>
   </xacro:macro>

Commit message: Fix wrist-branch transit planning and clean up repo
- NearestBranchTransitPlanner: plan free-space transits to the exact-pose,
  collision-free IK branch nearest the start state, so the corrected
  t_cut no longer winds joint6 (wrist guard unchanged).
- box_h_cut_executor: remove dead cut-debug planners and partial cut
  modes, merge cut-debug start into planCutSegments (now wrist-guarded),
  default cut_pattern t_cut, validate motion_profile at runtime, gate
  expensive left roll diagnostics behind a parameter.
- Transit scaling 0.15 (operator-approved); contact strokes unchanged.
- Remove box_motion_executor, rebel_mtc_ptp_lin, point_target_moveit,
  compare_detection, broken Setup Assistant launches, unused configs,
  dead CRI driver code, and the proposed-TCP marker link.
- Gamepad node loads gamepad.yaml and is named servo_gamepad_input.
- Docs, CLAUDE.md, .gitignore and .dockerignore updated.

Mock regression: target poses identical before/after for t_cut,
t_cut_handoff, h, combined, pilz profiles and cut-debug starts.

Co-Authored-By: Claude Opus 5.5 <noreply@anthropic.com>

File: src/igus_rebel_description/urdf/igus_rebel_xeg32_wrapper.urdf.xacro (robot description, xacro)
@@ -50,14 +50,3 @@
     <origin xyz="0.005937 0.094121 0.130699" rpy="0 0 0"/>
   </joint>
-  <link name="xeg32_tool_tip_proposed">
-    <visual>
-      <geometry><sphere radius="0.006"/></geometry>
-      <material name="xeg32_tool_tip_proposed_marker"><color rgba="1 0.1 0.1 1"/></material>
-    </visual>
-  </link>
-  <joint name="igus_tool0_to_xeg32_tool_tip_proposed" type="fixed">
-    <parent link="igus_tool0"/>
-    <child link="xeg32_tool_tip_proposed"/>
-    <origin xyz="0.088936 0.046766 0.135060" rpy="0 0 0"/>
-  </joint>
 </robot>

Commit message: Add collision geometry for XEG-32 gripper-mounted tooling
Model the ultrasonic knife handpiece, its holder (from JK-Final version.step)
and the wrist camera + bracket (estimated from photos, no CAD) as fixed links
off igus_tool0, with collision meshes in
igus_rebel_description/meshes/xeg32_collision/ and simple visuals; add them to
the xeg32_gripper SRDF group/end-effector and regenerate the self-collision
matrix (computeDefaultCollisions, matching the 2026-09-27 methodology). The
exposed ~20 mm of blade below the TCP is left uncollided, matching
xeg32_tool_tip, since it must contact the carton to cut; the H-cut executor's
scoped tool/carton contact allowance only ever applies to xeg32_tool_tip, so
the new links are never exempted from carton collision checking.

Mock-only regression (scan_results/tool_collision_20260928/) shows the knife
handpiece and holder introduce no regressions, but the wrist camera collides
with detected_carton/camera_pole for most cut patterns on the recorded replay
carton given the H-cut executor's tight approach clearances -- a genuine,
previously invisible reach conflict that needs the operator's attention before
running H-cut with a wrist camera physically mounted (see
XEG32_MOVEIT_CHANGES.md and HANDOFF.md).

Co-Authored-By: Claude Opus 5.5 <noreply@anthropic.com>

File: src/igus_rebel_description/urdf/igus_rebel_xeg32_wrapper.urdf.xacro (robot description, xacro)
@@ -53,3 +53,70 @@
     <origin xyz="0.005937 0.094121 0.130699" rpy="0 0 0"/>
   </joint>
+  <!-- Tooling mounted on the XEG-32 gripper (2026-09-28): the ultrasonic knife
+       handpiece + holder and the wrist camera + bracket. Collision-only
+       conservative hulls, registered from operator-confirmed measurements and
+       the JK-Final version.step CAD (handpiece, holder) or estimated from
+       photos scaled against the gripper (wrist camera); see
+       XEG32_MOVEIT_CHANGES.md and HANDOFF.md for the placement reasoning.
+       xeg32_tool_tip itself (the TCP, the exposed ~20 mm of blade below it)
+       intentionally carries no collision geometry. All origins here are
+       identity: the meshes are already expressed in igus_tool0 coordinates. -->
+  <xacro:if value="$(arg attach_xeg32)">
+    <link name="xeg32_knife_handpiece">
+      <visual>
+        <geometry><mesh filename="package://igus_rebel_description/meshes/xeg32_collision/knife_handpiece.stl"/></geometry>
+        <material name="xeg32_knife_handpiece_material"><color rgba="0.2 0.2 0.2 0.6"/></material>
+      </visual>
+      <collision>
+        <geometry><mesh filename="package://igus_rebel_description/meshes/xeg32_collision/knife_handpiece.stl"/></geometry>
+      </collision>
+    </link>
+    <joint name="igus_tool0_to_xeg32_knife_handpiece" type="fixed">
+      <parent link="igus_tool0"/>
+      <child link="xeg32_knife_handpiece"/>
+      <origin xyz="0 0 0" rpy="0 0 0"/>
+    </joint>
+    <link name="xeg32_knife_holder">
+      <visual>
+        <geometry><mesh filename="package://igus_rebel_description/meshes/xeg32_collision/knife_holder_ring.stl"/></geometry>
+        <material name="xeg32_knife_holder_material"><color rgba="0.6 0.6 0.6 0.6"/></material>
+      </visual>
+      <collision>
+        <geometry><mesh filename="package://igus_rebel_description/meshes/xeg32_collision/knife_holder_ring.stl"/></geometry>
+      </collision>
+      <visual>
+        <geometry><mesh filename="package://igus_rebel_description/meshes/xeg32_collision/knife_holder_body.stl"/></geometry>
+        <material name="xeg32_knife_holder_material"/>
+      </visual>
+      <collision>
+        <geometry><mesh filename="package://igus_rebel_description/meshes/xeg32_collision/knife_holder_body.stl"/></geometry>
+      </collision>
+    </link>
+    <joint name="igus_tool0_to_xeg32_knife_holder" type="fixed">
+      <parent link="igus_tool0"/>
+      <child link="xeg32_knife_holder"/>
+      <origin xyz="0 0 0" rpy="0 0 0"/>
+    </joint>
+    <link name="xeg32_wrist_camera">
+      <visual>
+        <geometry><mesh filename="package://igus_rebel_description/meshes/xeg32_collision/wrist_camera_bracket.stl"/></geometry>
+        <material name="xeg32_wrist_camera_material"><color rgba="0.1 0.1 0.1 0.6"/></material>
+      </visual>
+      <collision>
+        <geometry><mesh filename="package://igus_rebel_description/meshes/xeg32_collision/wrist_camera_bracket.stl"/></geometry>
+      </collision>
+      <visual>
+        <geometry><mesh filename="package://igus_rebel_description/meshes/xeg32_collision/wrist_camera_body.stl"/></geometry>
+        <material name="xeg32_wrist_camera_material"/>
+      </visual>
+      <collision>
+        <geometry><mesh filename="package://igus_rebel_description/meshes/xeg32_collision/wrist_camera_body.stl"/></geometry>
+      </collision>
+    </link>
+    <joint name="igus_tool0_to_xeg32_wrist_camera" type="fixed">
+      <parent link="igus_tool0"/>
+      <child link="xeg32_wrist_camera"/>
+      <origin xyz="0 0 0" rpy="0 0 0"/>
+    </joint>
+  </xacro:if>
 </robot>

Commit message: Remove wrist camera collision link; camera uninstalled for the holder redesign
The camera protruded past the blade tip along the knife axis and made
nearly every H-cut plan collide with the carton. The operator uninstalled
it until the combined knife/camera holder is redesigned. Knife handpiece
and holder collision geometry stay. Mock regression without the camera
matches the pre-tooling results, including parallel left mode.

Co-Authored-By: Claude Opus 5.5 <noreply@anthropic.com>

File: src/igus_rebel_description/urdf/igus_rebel_xeg32_wrapper.urdf.xacro (robot description, xacro)
@@ -98,25 +98,7 @@
       <origin xyz="0 0 0" rpy="0 0 0"/>
     </joint>
-    <link name="xeg32_wrist_camera">
-      <visual>
-        <geometry><mesh filename="package://igus_rebel_description/meshes/xeg32_collision/wrist_camera_bracket.stl"/></geometry>
-        <material name="xeg32_wrist_camera_material"><color rgba="0.1 0.1 0.1 0.6"/></material>
-      </visual>
-      <collision>
-        <geometry><mesh filename="package://igus_rebel_description/meshes/xeg32_collision/wrist_camera_bracket.stl"/></geometry>
-      </collision>
-      <visual>
-        <geometry><mesh filename="package://igus_rebel_description/meshes/xeg32_collision/wrist_camera_body.stl"/></geometry>
-        <material name="xeg32_wrist_camera_material"/>
-      </visual>
-      <collision>
-        <geometry><mesh filename="package://igus_rebel_description/meshes/xeg32_collision/wrist_camera_body.stl"/></geometry>
-      </collision>
-    </link>
-    <joint name="igus_tool0_to_xeg32_wrist_camera" type="fixed">
-      <parent link="igus_tool0"/>
-      <child link="xeg32_wrist_camera"/>
-      <origin xyz="0 0 0" rpy="0 0 0"/>
-    </joint>
+    <!-- Wrist camera removed 2026-09-28: it protruded past the blade tip along the knife
+         axis and hit the carton; it is uninstalled until the combined knife/camera holder
+         is redesigned. -->
   </xacro:if>
 </robot>
