Commit message: Harden CRI driver, executor safety gates and MoveIt config
CRI driver (igus_rebel):
- 50 ms stale-write watchdog zeroes ALIVEJOG; jog clamped to +/-100 %,
  NaN -> 0; on_deactivate/on_error zero the jog.
- Send Override 100.0 after MotionTypeJoint on every connect.
- Wait for the first valid STATUS before reporting state; read()
  fails closed on STATUS older than 200 ms or after any reconnect.
- Fix fd leak, split-frame loss (new CriFrameParser), parser crashes,
  data races, busy wait, shutdown hang; DIO service off the RT loop.
- JTC path/goal tolerances, D gains 0; unused velocity controller removed.
- New gtests incl. a fake CRI server on loopback.

box_h_cut_executor:
- Fix parameter-callback deadlock; runtime-ignored params read-only;
  stale-snapshot override blocks every execute; finite checks.
- Wrist guard fails closed on transit-count mismatch.
- Transit planner retries the pose goal once within one time budget.
- t_cut_handoff search probes 0.95 first and reuses the roll search.
- Scalings rescaled for the new joint limits (same physical speed).

MoveIt config:
- Joint limits 0.785 rad/s, 5.24 rad/s^2 (igus/CPR); Pilz cartesian
  limits rescaled; allowed_start_tolerance 0.02.
- SRDF collision matrix regenerated (100k samples).
- run_teleop default false; teleop calls start_servo on Humble;
  camera pole re-applied and clean shutdown; sim uses the XEG wrapper.

Other: perception one-shot filters removed, 1 s frame age; hand-eye
replay refuses to run without a TTY; decimated meshes and convex
carriage collision mesh; colcon test runs pytest; calibration default
rebel_handeye_h_v2; left correction default is the taught-angle record;
Dockerfile defaults to Humble; docs and HANDOFF rewritten.

Verified in mock/sim only: clean build with no warnings, 146 tests pass,
17-scenario planning regression matches baseline. Not yet run on the
real robot; see HANDOFF.md first-run checklist.

Co-Authored-By: Claude Opus 5.5 <noreply@anthropic.com>

File: src/igus_rebel_description/urdf/igus_rebel2.urdf (robot description, URDF)
Before this commit: robot igus_rebel, 12 links, 11 joints
Links:
- link base_link: geometry collision cylinder length=0.1 radius=0.09; visual mesh filename=package://igus_rebel_description/meshes/rebel_d00617809/bas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
- link link1: geometry collision box size=0.1 0.03 0.1; visual mesh filename=package://igus_rebel_description/meshes/rebel_d00617809/lin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
- link link2: geometry collision cylinder length=0.18 radius=0.06; visual mesh filename=package://igus_rebel_description/meshes/rebel_d00617809/lin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
- link link3: geometry collision box size=0.1 0.03 0.1; visual mesh filename=package://igus_rebel_description/meshes/rebel_d00617809/lin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
- link link4: geometry collision cylinder length=0.1 radius=0.05; visual mesh filename=package://igus_rebel_description/meshes/rebel_d00617809/lin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
- link link5: geometry collision box size=0.1 0.03 0.1; visual mesh filename=package://igus_rebel_description/meshes/rebel_d00617809/lin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
- link link6: geometry collision cylinder length=0.065 radius=0.04; visual mesh filename=package://igus_rebel_description/meshes/rebel_d00617809/lin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
- link motor1: geometry collision cylinder length=0.065 radius=0.05; visual mesh filename=package://igus_rebel_description/meshes/rebel_d00617809/mot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
- link motor2: geometry collision cylinder length=0.065 radius=0.05; visual mesh filename=package://igus_rebel_description/meshes/rebel_d00617809/mot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
- link motor3: geometry collision cylinder length=0.065 radius=0.05; visual mesh filename=package://igus_rebel_description/meshes/rebel_d00617809/mot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
- link motor4: geometry collision cylinder length=0.065 radius=0.05; visual mesh filename=package://igus_rebel_description/meshes/rebel_d00617809/mot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
- link motor5: geometry collision cylinder length=0.065 radius=0.04; visual mesh filename=package://igus_rebel_description/meshes/rebel_d00617809/mot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
Joints:
- joint joint1: limit lower=-3.1241 upper=3.1241 effort=330 velocity=2.16 -> lower=-3.1241 upper=3.1241 effort=330 velocity=0.785
- joint joint2: limit lower=-1.4835 upper=2.4435 effort=330 velocity=2.16 -> lower=-1.4835 upper=2.4435 effort=330 velocity=0.785
- joint joint3: limit lower=-1.39626 upper=2.61799 effort=330 velocity=2.16 -> lower=-1.39626 upper=2.61799 effort=330 velocity=0.785
- joint joint4: limit lower=-3.12414 upper=3.12414 effort=330 velocity=2.16 -> lower=-3.12414 upper=3.12414 effort=330 velocity=0.785
- joint joint5: limit lower=-1.65806 upper=1.65806 effort=330 velocity=2.16 -> lower=-1.65806 upper=1.65806 effort=330 velocity=0.785
- joint joint6: limit lower=-3.12414 upper=3.12414 effort=330 velocity=2.16 -> lower=-3.12414 upper=3.12414 effort=330 velocity=0.785

File: src/igus_rebel_description/urdf/xeg32_gripper.urdf.xacro (robot description, xacro)
@@ -1,5 +1,7 @@
 <?xml version='1.0' encoding='utf-8'?>
 <robot xmlns:xacro="http://www.ros.org/wiki/xacro">
-  <!-- Rough HIWIN XEG-32 gripper geometry; independent of TCP calibration. -->
+  <!-- Rough HIWIN XEG-32 gripper geometry; independent of TCP calibration.
+       Collision meshes in meshes/xeg32_collision/ are convex hulls of the
+       matching visual meshes (conservative, bounding boxes identical). -->
   <xacro:macro name="xeg32_gripper" params="parent_link prefix flange_xyz flange_rpy lock_joints:=true">
     <joint name="${prefix}mount_joint" type="fixed">
@@ -78,5 +80,5 @@
         <origin xyz="0 0.005 -0.0135" rpy="-3.14159 -0 -0" />
         <geometry>
-          <mesh filename="package://igus_rebel_description/meshes/xeg32/right_carriage.stl" />
+          <mesh filename="package://igus_rebel_description/meshes/xeg32_collision/right_carriage.stl" />
         </geometry>
       </collision>
@@ -130,5 +132,5 @@
         <origin xyz="0 0.005 -0.0135" rpy="-3.14159 0 0" />
         <geometry>
-          <mesh filename="package://igus_rebel_description/meshes/xeg32/right_carriage.stl" />
+          <mesh filename="package://igus_rebel_description/meshes/xeg32_collision/right_carriage.stl" />
         </geometry>
       </collision>

Commit message: Set joint limits from the real controller; add CRI limit query tool
The ReBeL controller (REBEL-6DOF-03) reports A2 -80..140 and A3 -80..140
deg, but the URDF allowed A2 down to -85 and A3 up to 150: a slider move
to 145 deg was stopped by the controller at 140. All six URDF limits now
sit 1 deg inside the controller limits. tools/cri_query_limits.py reads
them over CRI (read-only). h-pattern approach joint5 94.37 -> 94.0.

Mock regression: nominal t_cut/handoff/h/combined/Pilz/cut-debug plans
unchanged; the taught-angle left correction is now infeasible on the
replay carton (it needed joint3 ~141 deg, beyond the controller limit).

Co-Authored-By: Claude Opus 5.5 <noreply@anthropic.com>

File: src/igus_rebel_description/urdf/igus_rebel2.urdf (robot description, URDF)
Before this commit: robot igus_rebel, 12 links, 11 joints
Joints:
- joint joint1: limit lower=-3.1241 upper=3.1241 effort=330 velocity=0.785 -> lower=-3.106686 upper=3.106686 effort=330 velocity=0.785
- joint joint2: limit lower=-1.4835 upper=2.4435 effort=330 velocity=0.785 -> lower=-1.378810 upper=2.426008 effort=330 velocity=0.785
- joint joint3: limit lower=-1.39626 upper=2.61799 effort=330 velocity=0.785 -> lower=-1.378810 upper=2.426008 effort=330 velocity=0.785
- joint joint4: limit lower=-3.12414 upper=3.12414 effort=330 velocity=0.785 -> lower=-3.106686 upper=3.106686 effort=330 velocity=0.785
- joint joint5: limit lower=-1.65806 upper=1.65806 effort=330 velocity=0.785 -> lower=-1.640609 upper=1.640609 effort=330 velocity=0.785
- joint joint6: limit lower=-3.12414 upper=3.12414 effort=330 velocity=0.785 -> lower=-3.106686 upper=3.106686 effort=330 velocity=0.785
